Commit message: increased weight of base to prevent tipping

File: movo_common/movo_description/urdf/movo_components/movo_base.urdf.xacro (robot description, xacro)
@@ -45,5 +45,5 @@
         <link name="base_chassis_link">
 			<inertial>
-				<mass value="44.2877" />
+				<mass value="100.00" /> <!-- 44.2877 -->
 				<origin xyz="-0.009506 -0.013039 0.032319" />
 				<inertia ixx="0.000165"  ixy="0" ixz="0"

Commit message: adjustments in movo mass

File: movo_common/movo_description/urdf/movo_components/movo_base.urdf.xacro (robot description, xacro)
@@ -45,5 +45,5 @@
         <link name="base_chassis_link">
 			<inertial>
-				<mass value="100.00" /> <!-- 44.2877 -->
+				<mass value="140.00" /> <!-- 44.2877 -->
 				<origin xyz="-0.009506 -0.013039 0.032319" />
 				<inertia ixx="0.000165"  ixy="0" ixz="0"

File: movo_common/movo_description/urdf/movo_components/movo_body.urdf.xacro (robot description, xacro)
@@ -59,5 +59,5 @@
         <link name="upper_body_link">
 			<inertial>
-				<mass value="6.246912" />
+				<mass value="0.0" /> <!-- 6.246912 -->
 				<origin xyz="-0.080608 0.000290 0.286026" />
 				<inertia ixx="0.425973"  ixy="0.000022" ixz="-0.015916"
